File: kiCad_stuff/AS5600_I2C_v1/AS5600_I2C_v1.sch (KiCad schematic (older format))
At the start: 8 parts, among them J1 Conn_01x04, U1 AS5600_ASOM_v1

Commit message: Added proj footptint symbol lib with 2 user-made footprints
Parts:
- removed MH_BL1, MH_BR1, MH_TL1, MH_TR1: MountingHole, MountingHole:MountingHole_2.5mm_Pad, symbol Mechanical:MountingHole
- J1: footprint Connector_PinHeader_1.00mm:PinHeader_1x04_P1.00mm_Vertical -> modular_segment_PCB_footprints:EthernetWireConnectors_1x04_P2.00mm_1mmDiam
Changed lines of the file:
@@
 F 1 "AS5600_ASOM_v1" H 5250 4874 50  0000 C CNN
 F 2 "Package_SO:SOIC-8_3.9x4.9mm_P1.27mm" H 5200 3900 50  0001 C CNN
-F 3 "" H 5200 3900 50  0001 C CNN
+F 3 "~" H 5200 3900 50  0001 C CNN
 	1    5200 4100
 	1    0    0    -1
@@
 F 1 "100nF" H 4100 3750 39  0000 L CNN
 F 2 "Capacitor_SMD:C_0805_2012Metric" H 4400 3750 50  0001 C CNN
-F 3 "" H 4400 3750 50  0001 C CNN
+F 3 "~" H 4400 3750 50  0001 C CNN
 	1    4400 3750
 	1    0    0    -1
@@
 F 1 "1uF" H 4700 3750 39  0000 L CNN
 F 2 "Capacitor_SMD:C_0805_2012Metric" H 4600 3750 50  0001 C CNN
-F 3 "" H 4600 3750 50  0001 C CNN
+F 3 "~" H 4600 3750 50  0001 C CNN
 	1    4600 3750
 	1    0    0    -1
@@
 F 0 "J1" H 6630 3142 50  0000 L CNN
 F 1 "Conn_01x04" H 6630 3051 50  0000 L CNN
-F 2 "Connector_PinHeader_1.00mm:PinHeader_1x04_P1.00mm_Vertical" H 6550 3150 50  0001 C CNN
-F 3 "" H 6550 3150 50  0001 C CNN
+F 2 "modular_segment_PCB_footprints:EthernetWireConnectors_1x04_P2.00mm_1mmDiam" H 6550 3150 50  0001 C CNN
+F 3 "~" H 6550 3150 50  0001 C CNN
 	1    6550 3150
 	1    0    0    -1
@@
 Wire Wire Line
 	6250 3050 6350 3050
-$Comp
-L Mechanical:MountingHole MH_TL1
-U 1 1 5C1571F3
-P 4400 2650
-F 0 "MH_TL1" H 4500 2696 50  0000 L CNN
-F 1 "MountingHole" H 4500 2605 50  0000 L CNN
-F 2 "MountingHole:MountingHole_2.5mm_Pad" H 4400 2650 50  0001 C CNN
-F 3 "~" H 4400 2650 50  0001 C CNN
-	1    4400 2650
-	1    0    0    -1
-$EndComp
-$Comp
-L Mechanical:MountingHole MH_TR1
-U 1 1 5C15727F
-P 5350 2650
-F 0 "MH_TR1" H 5450 2696 50  0000 L CNN
-F 1 "MountingHole" H 5450 2605 50  0000 L CNN
-F 2 "MountingHole:MountingHole_2.5mm_Pad" H 5350 2650 50  0001 C CNN
-F 3 "~" H 5350 2650 50  0001 C CNN
-	1    5350 2650
-	1    0    0    -1
-$EndComp
-$Comp
-L Mechanical:MountingHole MH_BL1
-U 1 1 5C157343
-P 4400 4400
-F 0 "MH_BL1" H 4500 4446 50  0000 L CNN
-F 1 "MountingHole" H 4500 4355 50  0000 L CNN
-F 2 "MountingHole:MountingHole_2.5mm_Pad" H 4400 4400 50  0001 C CNN
-F 3 "~" H 4400 4400 50  0001 C CNN
-	1    4400 4400
-	1    0    0    -1
-$EndComp
-$Comp
-L Mechanical:MountingHole MH_BR1
-U 1 1 5C1573A5
-P 5450 4400
-F 0 "MH_BR1" H 5550 4446 50  0000 L CNN
-F 1 "MountingHole" H 5550 4355 50  0000 L CNN
-F 2 "MountingHole:MountingHole_2.5mm_Pad" H 5450 4400 50  0001 C CNN
-F 3 "~" H 5450 4400 50  0001 C CNN
-	1    5450 4400
-	1    0    0    -1
-$EndComp
 $EndSCHEMATC

Commit message: Ethernet-cable direct solder v2 completed
Changed lines of the file:
@@
 L Connector_Generic:Conn_01x04 J1
 U 1 1 5C155E4C
-P 6550 3150
-F 0 "J1" H 6630 3142 50  0000 L CNN
-F 1 "Conn_01x04" H 6630 3051 50  0000 L CNN
-F 2 "modular_segment_PCB_footprints:EthernetWireConnectors_1x04_P2.00mm_1mmDiam" H 6550 3150 50  0001 C CNN
-F 3 "~" H 6550 3150 50  0001 C CNN
-	1    6550 3150
-	1    0    0    -1
+P 6900 3250
+F 0 "J1" H 6980 3242 50  0000 L CNN
+F 1 "Conn_01x04" H 6980 3151 50  0000 L CNN
+F 2 "modular_segment_PCB_footprints:EthernetWireConnectors_1x04_P2.00mm_1mmDiam" H 6900 3250 50  0001 C CNN
+F 3 "~" H 6900 3250 50  0001 C CNN
+	1    6900 3250
+	-1   0    0    1
 $EndComp
 $Comp
 L power:+5V #PWR04
 U 1 1 5C155EA8
-P 6300 2950
-F 0 "#PWR04" H 6300 2800 50  0001 C CNN
-F 1 "+5V" H 6315 3123 50  0000 C CNN
-F 2 "" H 6300 2950 50  0001 C CNN
-F 3 "" H 6300 2950 50  0001 C CNN
-	1    6300 2950
+P 7150 2750
+F 0 "#PWR04" H 7150 2600 50  0001 C CNN
+F 1 "+5V" H 7165 2923 50  0000 C CNN
+F 2 "" H 7150 2750 50  0001 C CNN
+F 3 "" H 7150 2750 50  0001 C CNN
+	1    7150 2750
 	1    0    0    -1
 $EndComp
@@
 L power:GND #PWR05
 U 1 1 5C155EBF
-P 6300 3500
-F 0 "#PWR05" H 6300 3250 50  0001 C CNN
-F 1 "GND" H 6305 3327 50  0000 C CNN
-F 2 "" H 6300 3500 50  0001 C CNN
-F 3 "" H 6300 3500 50  0001 C CNN
-	1    6300 3500
+P 7150 3500
+F 0 "#PWR05" H 7150 3250 50  0001 C CNN
+F 1 "GND" H 7155 3327 50  0000 C CNN
+F 2 "" H 7150 3500 50  0001 C CNN
+F 3 "" H 7150 3500 50  0001 C CNN
+	1    7150 3500
 	1    0    0    -1
 $EndComp
-Wire Wire Line
-	6300 3500 6300 3250
-Wire Wire Line
-	6300 3250 6350 3250
-Wire Wire Line
-	6300 2950 6300 3150
-Wire Wire Line
-	6300 3150 6350 3150
-Text GLabel 6250 3050 0    50   Input ~ 0
+Text GLabel 7200 3050 2    50   Input ~ 0
 SDA
-Text GLabel 6250 3350 0    50   Input ~ 0
+Text GLabel 7200 3350 2    50   Input ~ 0
 SCL
 Wire Wire Line
-	6250 3350 6350 3350
+	7200 3350 7100 3350
 Wire Wire Line
-	6250 3050 6350 3050
+	7200 3050 7100 3050
+Wire Wire Line
+	7150 3150 7100 3150
+Wire Wire Line
+	7150 2750 7150 3150
+Wire Wire Line
+	7150 3250 7150 3500
+Wire Wire Line
+	7100 3250 7150 3250
 $EndSCHEMATC
