File: kiCad_stuff/AS5600_I2C_eth_v2/AS5600_I2C_v1.sch (KiCad schematic (older format))
At the start: 4 parts, among them J1 Conn_01x04, U1 AS5600_ASOM_v1

Commit message: Started designing PCB using ADC-to-I2C chip
Parts:
- added U2: MCP3221, Package_TO_SOT_SMD:SOT-23-5, symbol AS5600_ASOM_AIWilmot:MCP3221
- U1: symbol modular_segment_lib:AS5600_ASOM_v1 -> AS5600_ASOM_AIWilmot:AS5600_ASOM_v1
Connections:
- net labels added: ANALOG
- wire segments 21 -> 28
- no-connect marks 0 -> 3
Changed lines of the file:
@@
 EESchema Schematic File Version 4
+LIBS:AS5600_I2C_v1-cache
 EELAYER 26 0
 EELAYER END
@@
 $EndDescr
 $Comp
-L modular_segment_lib:AS5600_ASOM_v1 U1
-U 1 1 5C1543A2
-P 5200 4100
-F 0 "U1" H 5250 4965 50  0000 C CNN
-F 1 "AS5600_ASOM_v1" H 5250 4874 50  0000 C CNN
-F 2 "Package_SO:SOIC-8_3.9x4.9mm_P1.27mm" H 5200 3900 50  0001 C CNN
-F 3 "~" H 5200 3900 50  0001 C CNN
-	1    5200 4100
-	1    0    0    -1
-$EndComp
-$Comp
 L Device:C C1
 U 1 1 5C1544B6
-P 4400 3750
-F 0 "C1" H 4300 3850 50  0000 L CNN
-F 1 "100nF" H 4100 3750 39  0000 L CNN
-F 2 "Capacitor_SMD:C_0805_2012Metric" H 4400 3750 50  0001 C CNN
-F 3 "~" H 4400 3750 50  0001 C CNN
-	1    4400 3750
-	1    0    0    -1
-$EndComp
-$Comp
-L Device:C C2
-U 1 1 5C154617
-P 4600 3750
-F 0 "C2" H 4600 3850 50  0000 L CNN
-F 1 "1uF" H 4700 3750 39  0000 L CNN
-F 2 "Capacitor_SMD:C_0805_2012Metric" H 4600 3750 50  0001 C CNN
-F 3 "~" H 4600 3750 50  0001 C CNN
-	1    4600 3750
+P 4300 3800
+F 0 "C1" H 4100 3800 50  0000 L CNN
+F 1 "100nF" H 4100 3700 39  0000 L CNN
+F 2 "Capacitor_SMD:C_0805_2012Metric" H 4300 3800 50  0001 C CNN
+F 3 "~" H 4300 3800 50  0001 C CNN
+	1    4300 3800
 	1    0    0    -1
 $EndComp
@@
 L power:GND #PWR03
 U 1 1 5C154838
-P 5650 3950
-F 0 "#PWR03" H 5650 3700 50  0001 C CNN
-F 1 "GND" H 5655 3777 50  0000 C CNN
-F 2 "" H 5650 3950 50  0001 C CNN
-F 3 "" H 5650 3950 50  0001 C CNN
-	1    5650 3950
+P 5650 4000
+F 0 "#PWR03" H 5650 3750 50  0001 C CNN
+F 1 "GND" H 5655 3827 50  0000 C CNN
+F 2 "" H 5650 4000 50  0001 C CNN
+F 3 "" H 5650 4000 50  0001 C CNN
+	1    5650 4000
 	1    0    0    -1
 $EndComp
@@
 	4900 3800 4850 3800
 Wire Wire Line
-	4850 3800 4850 3950
-Wire Wire Line
-	4900 3600 4600 3600
-Wire Wire Line
-	4400 3600 4400 3500
-Wire Wire Line
-	4400 3500 4900 3500
-Wire Wire Line
-	4400 3900 4400 3950
-Wire Wire Line
-	4400 3950 4600 3950
-Connection ~ 4850 3950
-Wire Wire Line
-	4850 3950 4850 4000
-Wire Wire Line
-	4600 3900 4600 3950
-Connection ~ 4600 3950
-Wire Wire Line
-	4600 3950 4850 3950
-Wire Wire Line
 	5600 3500 5650 3500
-Text GLabel 5750 3700 2    50   Input ~ 0
-SDA
-Text GLabel 5750 3600 2    50   Input ~ 0
-SCL
-Wire Wire Line
-	5600 3600 5750 3600
-Wire Wire Line
-	5600 3700 5750 3700
-Wire Wire Line
-	5650 3500 5650 3950
 $Comp
 L power:+5V #PWR01
 U 1 1 5C155410
-P 4400 3400
-F 0 "#PWR01" H 4400 3250 50  0001 C CNN
-F 1 "+5V" H 4415 3573 50  0000 C CNN
-F 2 "" H 4400 3400 50  0001 C CNN
-F 3 "" H 4400 3400 50  0001 C CNN
-	1    4400 3400
-	1    0    0    -1
-$EndComp
-Wire Wire Line
-	4400 3400 4400 3500
-Connection ~ 4400 3500
+P 4300 3400
+F 0 "#PWR01" H 4300 3250 50  0001 C CNN
+F 1 "+5V" H 4315 3573 50  0000 C CNN
+F 2 "" H 4300 3400 50  0001 C CNN
+F 3 "" H 4300 3400 50  0001 C CNN
+	1    4300 3400
+	1    0    0    -1
+$EndComp
 $Comp
 L Connector_Generic:Conn_01x04 J1
 U 1 1 5C155E4C
-P 6900 3250
-F 0 "J1" H 6980 3242 50  0000 L CNN
-F 1 "Conn_01x04" H 6980 3151 50  0000 L CNN
-F 2 "modular_segment_PCB_footprints:EthernetWireConnectors_1x04_P2.00mm_1mmDiam" H 6900 3250 50  0001 C CNN
-F 3 "~" H 6900 3250 50  0001 C CNN
-	1    6900 3250
+P 6350 3750
+F 0 "J1" H 6300 3450 50  0000 L CNN
+F 1 "Conn_01x04" H 6300 3350 50  0000 L CNN
+F 2 "modular_segment_PCB_footprints:EthernetWireConnectors_1x04_P2.00mm_1mmDiam" H 6350 3750 50  0001 C CNN
+F 3 "~" H 6350 3750 50  0001 C CNN
+	1    6350 3750
 	-1   0    0    1
 $EndComp
@@
 L power:+5V #PWR04
 U 1 1 5C155EA8
-P 7150 2750
-F 0 "#PWR04" H 7150 2600 50  0001 C CNN
-F 1 "+5V" H 7165 2923 50  0000 C CNN
-F 2 "" H 7150 2750 50  0001 C CNN
-F 3 "" H 7150 2750 50  0001 C CNN
-	1    7150 2750
+P 7000 3650
+F 0 "#PWR04" H 7000 3500 50  0001 C CNN
+F 1 "+5V" H 7015 3823 50  0000 C CNN
+F 2 "" H 7000 3650 50  0001 C CNN
+F 3 "" H 7000 3650 50  0001 C CNN
+	1    7000 3650
 	1    0    0    -1
 $EndComp
@@
 L power:GND #PWR05
 U 1 1 5C155EBF
-P 7150 3500
-F 0 "#PWR05" H 7150 3250 50  0001 C CNN
-F 1 "GND" H 7155 3327 50  0000 C CNN
-F 2 "" H 7150 3500 50  0001 C CNN
-F 3 "" H 7150 3500 50  0001 C CNN
-	1    7150 3500
-	1    0    0    -1
-$EndComp
-Text GLabel 7200 3050 2    50   Input ~ 0
+P 6600 3900
+F 0 "#PWR05" H 6600 3650 50  0001 C CNN
+F 1 "GND" H 6750 3850 50  0000 C CNN
+F 2 "" H 6600 3900 50  0001 C CNN
+F 3 "" H 6600 3900 50  0001 C CNN
+	1    6600 3900
+	1    0    0    -1
+$EndComp
+Text GLabel 6650 3550 2    50   Input ~ 0
 SDA
-Text GLabel 7200 3350 2    50   Input ~ 0
+Text GLabel 6650 3650 2    50   Input ~ 0
 SCL
-Wire Wire Line
-	7200 3350 7100 3350
-Wire Wire Line
-	7200 3050 7100 3050
-Wire Wire Line
-	7150 3150 7100 3150
-Wire Wire Line
-	7150 2750 7150 3150
-Wire Wire Line
-	7150 3250 7150 3500
-Wire Wire Line
-	7100 3250 7150 3250
+$Comp
+L AS5600_ASOM_AIWilmot:MCP3221 U2
+U 1 1 5C70752F
+P 3500 3250
+F 0 "U2" H 3600 3750 50  0000 C CNN
+F 1 "MCP3221" H 3600 3350 50  0000 C CNN
+F 2 "Package_TO_SOT_SMD:SOT-23-5" H 3500 3250 50  0001 C CNN
+F 3 "https://docs-emea.rs-online.com/webdocs/1380/0900766b81380b0c.pdf" H 3500 3250 50  0001 C CNN
+	1    3500 3250
+	-1   0    0    1
+$EndComp
+Text GLabel 3050 3500 0    50   Output ~ 0
+SDA
+Text GLabel 3050 3600 0    50   Output ~ 0
+SCL
+NoConn ~ 5600 3700
+NoConn ~ 5600 3600
+Wire Wire Line
+	3100 3600 3050 3600
+Wire Wire Line
+	3050 3500 3100 3500
+$Comp
+L AS5600_ASOM_AIWilmot:AS5600_ASOM_v1 U1
+U 1 1 5C1543A2
+P 5200 4100
+F 0 "U1" H 5250 4965 50  0000 C CNN
+F 1 "AS5600_ASOM_v1" H 5250 4874 50  0000 C CNN
+F 2 "Package_SO:SOIC-8_3.9x4.9mm_P1.27mm" H 5200 3900 50  0001 C CNN
+F 3 "https://www.mouser.com/pdfdocs/AMS_AS5600_Datasheet_EN.PDF" H 5200 3900 50  0001 C CNN
+	1    5200 4100
+	1    0    0    -1
+$EndComp
+Wire Wire Line
+	4500 3600 4500 3650
+$Comp
+L Device:C C2
+U 1 1 5C154617
+P 4500 3800
+F 0 "C2" H 4600 3800 50  0000 L CNN
+F 1 "1uF" H 4550 3700 39  0000 L CNN
+F 2 "Capacitor_SMD:C_0805_2012Metric" H 4500 3800 50  0001 C CNN
+F 3 "~" H 4500 3800 50  0001 C CNN
+	1    4500 3800
+	1    0    0    -1
+$EndComp
+Wire Wire Line
+	4300 3400 4300 3500
+Wire Wire Line
+	4300 3950 4500 3950
+Connection ~ 4500 3950
+Text GLabel 4850 3700 0    50   Output ~ 0
+ANALOG
+Wire Wire Line
+	4850 3800 4850 3950
+Wire Wire Line
+	4500 3950 4850 3950
+Connection ~ 4850 3950
+Wire Wire Line
+	4850 3950 4850 4000
+Wire Wire Line
+	4500 3600 4900 3600
+Wire Wire Line
+	4850 3700 4900 3700
+Wire Wire Line
+	4900 3500 4300 3500
+Connection ~ 4300 3500
+Wire Wire Line
+	4300 3500 4300 3650
+Text GLabel 3800 3450 2    50   Input ~ 0
+ANALOG
+Wire Wire Line
+	3700 3450 3800 3450
+Wire Wire Line
+	4300 3950 3850 3950
+Wire Wire Line
+	3850 3950 3850 3550
+Wire Wire Line
+	3850 3550 3700 3550
+Connection ~ 4300 3950
+Wire Wire Line
+	3700 3650 4200 3650
+Wire Wire Line
+	4200 3650 4200 3500
+Wire Wire Line
+	4200 3500 4300 3500
+Wire Wire Line
+	5650 3500 5650 4000
+NoConn ~ 5600 3800
+Wire Wire Line
+	6550 3650 6650 3650
+Wire Wire Line
+	6550 3550 6650 3550
+Wire Wire Line
+	7000 3750 7000 3650
+Wire Wire Line
+	6550 3850 6600 3850
+Wire Wire Line
+	6600 3850 6600 3900
+Wire Wire Line
+	6550 3750 7000 3750
 $EndSCHEMATC
