File: kiCad_stuff/AS5600_ANALOG_TO_I2C_v2/AS5600_I2C_v1.sch (KiCad schematic (older format))
At the start: 5 parts, among them J1 Conn_01x04, U1 AS5600_ASOM_v1, U2 MCP3221

Commit message: More slave-device addresses using ADC-to-I2C converter.
Parts:
- J1: footprint modular_segment_PCB_footprints:EthernetWireConnectors_1x04_P2.00mm_1mmDiam -> Connector_PinHeader_2.00mm:PinHeader_1x04_P2.00mm_Vertical
- U2: footprint Package_TO_SOT_SMD:SOT-23-5 -> Package_TO_SOT_SMD:SOT-23-5_HandSoldering
Connections:
- wire segments 28 -> 27
Changed lines of the file:
@@
 F 0 "J1" H 6300 3450 50  0000 L CNN
 F 1 "Conn_01x04" H 6300 3350 50  0000 L CNN
-F 2 "modular_segment_PCB_footprints:EthernetWireConnectors_1x04_P2.00mm_1mmDiam" H 6350 3750 50  0001 C CNN
-F 3 "~" H 6350 3750 50  0001 C CNN
+F 2 "Connector_PinHeader_2.00mm:PinHeader_1x04_P2.00mm_Vertical" H 6350 3750 50  0001 C CNN
+F 3 "https://docs-emea.rs-online.com/webdocs/0025/0900766b80025f11.pdf" H 6350 3750 50  0001 C CNN
 	1    6350 3750
 	-1   0    0    1
 $EndComp
 $Comp
-L power:+5V #PWR04
+L power:+5V #PWR05
 U 1 1 5C155EA8
-P 7000 3650
-F 0 "#PWR04" H 7000 3500 50  0001 C CNN
-F 1 "+5V" H 7015 3823 50  0000 C CNN
-F 2 "" H 7000 3650 50  0001 C CNN
-F 3 "" H 7000 3650 50  0001 C CNN
-	1    7000 3650
+P 6900 3450
+F 0 "#PWR05" H 6900 3300 50  0001 C CNN
+F 1 "+5V" H 7050 3500 50  0000 C CNN
+F 2 "" H 6900 3450 50  0001 C CNN
+F 3 "" H 6900 3450 50  0001 C CNN
+	1    6900 3450
 	1    0    0    -1
 $EndComp
 $Comp
-L power:GND #PWR05
+L power:GND #PWR04
 U 1 1 5C155EBF
-P 6600 3900
-F 0 "#PWR05" H 6600 3650 50  0001 C CNN
+P 6650 3850
+F 0 "#PWR04" H 6650 3600 50  0001 C CNN
 F 1 "GND" H 6750 3850 50  0000 C CNN
-F 2 "" H 6600 3900 50  0001 C CNN
-F 3 "" H 6600 3900 50  0001 C CNN
-	1    6600 3900
+F 2 "" H 6650 3850 50  0001 C CNN
+F 3 "" H 6650 3850 50  0001 C CNN
+	1    6650 3850
 	1    0    0    -1
 $EndComp
@@
 F 0 "U2" H 3600 3750 50  0000 C CNN
 F 1 "MCP3221" H 3600 3350 50  0000 C CNN
-F 2 "Package_TO_SOT_SMD:SOT-23-5" H 3500 3250 50  0001 C CNN
+F 2 "Package_TO_SOT_SMD:SOT-23-5_HandSoldering" H 3500 3250 50  0001 C CNN
 F 3 "https://docs-emea.rs-online.com/webdocs/1380/0900766b81380b0c.pdf" H 3500 3250 50  0001 C CNN
 	1    3500 3250
@@
 NoConn ~ 5600 3800
 Wire Wire Line
-	6550 3650 6650 3650
-Wire Wire Line
 	6550 3550 6650 3550
 Wire Wire Line
-	7000 3750 7000 3650
+	6650 3650 6550 3650
 Wire Wire Line
-	6550 3850 6600 3850
+	6900 3450 6900 3750
 Wire Wire Line
-	6600 3850 6600 3900
+	6900 3750 6550 3750
 Wire Wire Line
-	6550 3750 7000 3750
+	6550 3850 6650 3850
 $EndSCHEMATC
