File: kiCad_stuff/Current_sensing/Current_sensing_circuits.sch (KiCad schematic (older format))
At the start: 5 parts, among them J1 Conn_01x02, J2 Conn_01x03, U1 INA283

Commit message: Added company logo to PCB library
Parts:
- C_bypass1: footprint Capacitors_SMD:C_0805_HandSoldering -> Capacitors_SMD:C_0805; symbol C -> Device:C
- J1: footprint Pin_Headers:Pin_Header_Straight_1x02_Pitch2.00mm -> Connector_PinSocket_2.54mm:PinSocket_1x02_P2.54mm_Vertical; symbol Conn_01x02 -> Current_sensing_circuits-rescue:Conn_01x02
- J2: footprint Pin_Headers:Pin_Header_Straight_1x03_Pitch2.00mm -> Connector_PinSocket_2.54mm:PinSocket_1x03_P2.54mm_Vertical; symbol Conn_01x03 -> Current_sensing_circuits-rescue:Conn_01x03
- R_shunt1: footprint Resistors_SMD:R_2512_HandSoldering -> Resistors_SMD:R_2512; symbol R -> Device:R
- U1: symbol INA283 -> Current_sensing_circuits-rescue:INA283
Changed lines of the file:
@@
-EESchema Schematic File Version 2
-LIBS:power
-LIBS:device
-LIBS:switches
-LIBS:relays
-LIBS:motors
-LIBS:transistors
-LIBS:conn
-LIBS:linear
-LIBS:regul
-LIBS:74xx
-LIBS:cmos4000
-LIBS:adc-dac
-LIBS:memory
-LIBS:xilinx
-LIBS:microcontrollers
-LIBS:dsp
-LIBS:microchip
-LIBS:analog_switches
-LIBS:motorola
-LIBS:texas
-LIBS:intel
-LIBS:audio
-LIBS:interface
-LIBS:digital-audio
-LIBS:philips
-LIBS:display
-LIBS:cypress
-LIBS:siliconi
-LIBS:opto
-LIBS:atmel
-LIBS:contrib
-LIBS:valves
+EESchema Schematic File Version 4
 LIBS:Current_sensing_circuits-cache
-EELAYER 25 0
+EELAYER 26 0
 EELAYER END
 $Descr A4 11693 8268
@@
 $EndDescr
 $Comp
-L INA283 U1
+L Current_sensing_circuits-rescue:INA283 U1
 U 1 1 5C8900FA
 P 5900 3500
@@
 $EndComp
 $Comp
-L R R_shunt1
+L Device:R R_shunt1
 U 1 1 5C8901B3
 P 5350 3500
 F 0 "R_shunt1" V 5430 3500 50  0000 C CNN
 F 1 "0.02" V 5250 3500 50  0000 C CNN
-F 2 "Resistors_SMD:R_2512_HandSoldering" V 5280 3500 50  0001 C CNN
+F 2 "Resistors_SMD:R_2512" V 5280 3500 50  0001 C CNN
 F 3 "" H 5350 3500 50  0001 C CNN
 	1    5350 3500
@@
 PWR+
 Wire Wire Line
-	5350 3200 5350 3350
+	5350 3200 5350 3300
 Wire Wire Line
-	5350 3650 5350 3800
+	5350 3650 5350 3700
 Wire Wire Line
 	5600 3600 5600 3700
@@
 Connection ~ 5350 3300
 $Comp
-L C C_bypass1
+L Device:C C_bypass1
 U 1 1 5C890899
 P 6050 3100
 F 0 "C_bypass1" V 5900 3100 50  0000 L CNN
 F 1 "0.1u" H 6075 3000 50  0000 L CNN
-F 2 "Capacitors_SMD:C_0805_HandSoldering" H 6088 2950 50  0001 C CNN
+F 2 "Capacitors_SMD:C_0805" H 6088 2950 50  0001 C CNN
 F 3 "" H 6050 3100 50  0001 C CNN
 	1    6050 3100
@@
 	6000 3750 6000 3700
 $Comp
-L Conn_01x02 J1
+L Current_sensing_circuits-rescue:Conn_01x02 J1
 U 1 1 5C890FE5
 P 4900 3500
 F 0 "J1" H 4900 3600 50  0000 C CNN
 F 1 "Conn_01x02" H 4900 3300 50  0000 C CNN
-F 2 "Pin_Headers:Pin_Header_Straight_1x02_Pitch2.00mm" H 4900 3500 50  0001 C CNN
+F 2 "Connector_PinSocket_2.54mm:PinSocket_1x02_P2.54mm_Vertical" H 4900 3500 50  0001 C CNN
 F 3 "" H 4900 3500 50  0001 C CNN
 	1    4900 3500
@@
 $EndComp
 $Comp
-L Conn_01x03 J2
+L Current_sensing_circuits-rescue:Conn_01x03 J2
 U 1 1 5C891056
 P 7400 3500
 F 0 "J2" H 7400 3700 50  0000 C CNN
 F 1 "Conn_01x03" H 7400 3300 50  0000 C CNN
-F 2 "Pin_Headers:Pin_Header_Straight_1x03_Pitch2.00mm" H 7400 3500 50  0001 C CNN
+F 2 "Connector_PinSocket_2.54mm:PinSocket_1x03_P2.54mm_Vertical" H 7400 3500 50  0001 C CNN
 F 3 "" H 7400 3500 50  0001 C CNN
 	1    7400 3500
@@
 Wire Wire Line
 	7600 3500 7750 3500
+Wire Wire Line
+	5350 3700 5350 3800
+Wire Wire Line
+	5350 3300 5350 3350
 $EndSCHEMATC
