Commit message: making Gazebo launch file, and added dummy mass/ inertia values to successfully get robot model to spawn

File: urdf_stuff/src/mypackage/robot.urdf (robot description, URDF)
Before this commit: robot gummi, 4 links, 3 joints
Links:
- link base: mass 0 -> 0.01
- link link1: mass 0 -> 0.01
- link link2: mass 0 -> 0.01
