Commit message: Simulated 8-DOF segment in gazebo, PID controllers are tricky to tune; using XACRO to simplify URDF

File: urdf_stuff/src/sara_8dof_v1/SARA.urdf (robot description, URDF)
Before this commit: robot SARA, 4 links, 3 joints
Links:
- added link link10, mass 1.0; collision mesh filename=package://sara_8dof_v1/meshes/link1.stl; visual mesh filename=package://sara_8dof_v1/meshes/link1.stl
- added link link11, mass 1.0; collision mesh filename=package://sara_8dof_v1/meshes/link2.stl; visual mesh filename=package://sara_8dof_v1/meshes/link2.stl
- added link link3, mass 1.0; collision mesh filename=package://sara_8dof_v1/meshes/base_link.stl; visual mesh filename=package://sara_8dof_v1/meshes/base_link.stl
- added link link4, mass 1.0; collision mesh filename=package://sara_8dof_v1/meshes/link1.stl; visual mesh filename=package://sara_8dof_v1/meshes/link1.stl
- added link link5, mass 1.0; collision mesh filename=package://sara_8dof_v1/meshes/link2.stl; visual mesh filename=package://sara_8dof_v1/meshes/link2.stl
- added link link6, mass 1.0; collision mesh filename=package://sara_8dof_v1/meshes/base_link.stl; visual mesh filename=package://sara_8dof_v1/meshes/base_link.stl
- added link link7, mass 1.0; collision mesh filename=package://sara_8dof_v1/meshes/link1.stl; visual mesh filename=package://sara_8dof_v1/meshes/link1.stl
- added link link8, mass 1.0; collision mesh filename=package://sara_8dof_v1/meshes/link2.stl; visual mesh filename=package://sara_8dof_v1/meshes/link2.stl
- added link link9, mass 1.0; collision mesh filename=package://sara_8dof_v1/meshes/base_link.stl; visual mesh filename=package://sara_8dof_v1/meshes/base_link.stl
- link base_link: geometry collision mesh filename=package://sara_8dof_v1/meshes/base_link.stl; visual mesh filename=package://sara_8dof_v1/meshes/base_link.stl
Joints:
- added joint fourth_segment_base: type fixed, parent link8, child link9, origin xyz=-0.02661 0.025554 -0.0153545 rpy=0 0 0
- added joint joint2: type revolute, parent link3, child link4, origin xyz=0.0431603651232 0.0484824520656 0.0274545091047 rpy=0.0 0.0 0.0, axis -1.0 0.0 0.0, limit lower=-0.7853981633974483 upper=0.7853981633974483 effort=30 velocity=1.0
- added joint joint3: type revolute, parent link4, child link5, origin xyz=-0.01655 0.040054 -0.0121 rpy=0.0 0.0 0.0, axis 0.0 0.0 1.0, limit lower=-0.7853981633974483 upper=0.7853981633974483 effort=30 velocity=1.0
- added joint joint4: type revolute, parent link6, child link7, origin xyz=0.0431603651232 0.0484824520656 0.0274545091047 rpy=0.0 0.0 0.0, axis -1.0 0.0 0.0, limit lower=-0.7853981633974483 upper=0.7853981633974483 effort=30 velocity=1.0
- added joint joint5: type revolute, parent link7, child link8, origin xyz=-0.01655 0.040054 -0.0121 rpy=0.0 0.0 0.0, axis 0.0 0.0 1.0, limit lower=-0.7853981633974483 upper=0.7853981633974483 effort=30 velocity=1.0
- added joint joint6: type revolute, parent link9, child link10, origin xyz=0.0431603651232 0.0484824520656 0.0274545091047 rpy=0.0 0.0 0.0, axis -1.0 0.0 0.0, limit lower=-0.7853981633974483 upper=0.7853981633974483 effort=30 velocity=1.0
- added joint joint7: type revolute, parent link10, child link11, origin xyz=-0.01655 0.040054 -0.0121 rpy=0.0 0.0 0.0, axis 0.0 0.0 1.0, limit lower=-0.7853981633974483 upper=0.7853981633974483 effort=30 velocity=1.0
- added joint second_segment_base: type fixed, parent link2, child link3, origin xyz=-0.02661 0.025554 -0.0153545 rpy=0 0 0
- added joint third_segment_base: type fixed, parent link5, child link6, origin xyz=-0.02661 0.025554 -0.0153545 rpy=0 0 0
- joint joint0: axis -1.0000000000000036 8.979975634925549e-16 3.609607530446545e-15 -> -1.0 0.0 0.0; limit lower=-0.7853981633974483 upper=0.7853981633974483 effort=99 velocity=99 -> lower=-0.7853981633974483 upper=0.7853981633974483 effort=30 velocity=1.0; origin xyz=0.04316036512320408 0.04848245206563817 0.027454509104734993 rpy=0.0 0.0 0.0 -> xyz=0.0431603651232 0.0484824520656 0.0274545091047 rpy=0.0 0.0 0.0
- joint joint1: axis 5.267338778969267e-15 -5.467848396278865e-15 1.0000000000000524 -> 0.0 0.0 1.0; limit lower=-0.7853981633974483 upper=0.7853981633974483 effort=99 velocity=99 -> lower=-0.7853981633974483 upper=0.7853981633974483 effort=30 velocity=1.0; origin xyz=-0.016550000000000054 0.040054000000004225 -0.01210000000000057 rpy=0.0 0.0 0.0 -> xyz=-0.01655 0.040054 -0.0121 rpy=0.0 0.0 0.0
