Commit message: automating urdf gen by placing xacro params in launch files

File: urdf_stuff/src/sara_8dof_v1/SARA.urdf.xacro (robot description, xacro)
@@ -81,5 +81,5 @@
     <xacro:simple_link link_name="link5" stl_name="link2"/>
 	<joint name="second_segment_base" type="fixed">
-	    <origin rpy="0 0 0" xyz="-0.02661 ${joint_1_y-0.0145} -0.0153545"/>
+	    <origin rpy="0 0 0" xyz="-0.02661 ${joint_1_y-0.0145-0.005} -0.0153545"/>
 		<parent link="link2"/>
 		<child link="link3"/>
@@ -98,5 +98,5 @@
     <xacro:simple_link link_name="link8" stl_name="link2"/>
 	<joint name="third_segment_base" type="fixed">
-	    <origin rpy="0 0 0" xyz="-0.02661 ${joint_1_y-0.0145} -0.0153545"/>
+	    <origin rpy="0 0 0" xyz="-0.02661 ${joint_1_y-0.0145-0.005} -0.0153545"/>
 		<parent link="link5"/>
 		<child link="link6"/>
@@ -115,5 +115,5 @@
     <xacro:simple_link link_name="link11" stl_name="link2"/>
 	<joint name="fourth_segment_base" type="fixed">
-	    <origin rpy="0 0 0" xyz="-0.02661 ${joint_1_y-0.0145} -0.0153545"/>
+	    <origin rpy="0 0 0" xyz="-0.02661 ${joint_1_y-0.0145-0.005} -0.0153545"/>
 		<parent link="link8"/>
 		<child link="link9"/>

Commit message: added damping to prevent issues with joint jittering around axis in gazebo sim

File: urdf_stuff/src/sara_8dof_v1/SARA.urdf.xacro (robot description, xacro)
@@ -8,6 +8,6 @@
         <inertial>
             <origin rpy="0.0 0.0 0.0" xyz="0.0 0.0 0.0"/>
-            <mass value="1.0"/>
-            <inertia ixx="0.04" ixy="0.04" ixz="0.04" iyy="0.04" iyz="0.04" izz="0.04"/>
+            <mass value="0.2"/>
+            <inertia ixx="0.01" ixy="0.01" ixz="0.01" iyy="0.01" iyz="0.01" izz="0.01"/>
         </inertial>
         <visual>
@@ -27,4 +27,8 @@
         </collision>
     </link>
+    <!-- Slow down gazebo sim to prevent erratic behaviour (https://answers.ros.org/question/43429/making-revolute-joint-stay-at-rest-if-no-effortwrench-is-applied/)-->
+    <gazebo reference="${link_name}">
+        <dampingFactor>0.1</dampingFactor>
+    </gazebo>
     <!--*********************************************************************************-->
 </xacro:macro>
