Commit message: Getting display.launch

File: urdf_stuff/src/wheelchair/robot.urdf (robot description, URDF)
Before this commit: robot gummi, 4 links, 3 joints
Links:
- link base: geometry collision mesh filename=package://wheelchair/meshes/base.stl; visual mesh filename=package://wheelchair/meshes/base.stl
- link link1: geometry collision mesh filename=package://wheelchair/meshes/link1.stl; visual mesh filename=package://wheelchair/meshes/link1.stl
- link link2: geometry collision mesh filename=package://wheelchair/meshes/link2.stl; visual mesh filename=package://wheelchair/meshes/link2.stl
