Commit message: Added another segment to chain

File: urdf_stuff/src/wheelchair/robot.urdf.xacro (robot description, xacro)
@@ -221,4 +221,21 @@
         <axis xyz="0.0 0.0 1.0"/>
     </xacro:segment_joints>
+<!-- Fifth segment (test) -->
+    <xacro:simple_link link_name="link12" stl_name="segment_base"/>
+    <xacro:simple_link link_name="link13" stl_name="segment_link1"/>
+    <xacro:simple_link link_name="link14" stl_name="segment_link2"/>
+	<joint name="fifth_segment_base" type="fixed">
+	    <origin rpy="0 0 0" xyz="-0.02661 ${joint_1_y-0.0145-0.005} -0.0153545"/>
+		<parent link="link11"/>
+		<child link="link12"/>
+	</joint>
+    <xacro:segment_joints joint_num="8" parent_link="link12" child_link="link13">
+        <origin rpy="0.0 0.0 0.0" xyz="${joint_0_x} ${joint_0_y} ${joint_0_z}"/>
+        <axis xyz="-1.0 0.0 0.0"/>
+    </xacro:segment_joints>
+    <xacro:segment_joints joint_num="9" parent_link="link13" child_link="link14">
+        <origin rpy="0.0 0.0 0.0" xyz="${joint_1_x} ${joint_1_y} ${joint_1_z}"/>
+        <axis xyz="0.0 0.0 1.0"/>
+    </xacro:segment_joints>
 	<!--
 		 Gazebo plugins:

Commit message: lined-up rigid link with shoulder

File: urdf_stuff/src/wheelchair/robot.urdf.xacro (robot description, xacro)
@@ -154,13 +154,18 @@
 <xacro:property name="joint_1_z" value="-0.01210000000000057" />
 <!-- First segment -->
-    <xacro:simple_link link_name="link0" stl_name="segment_base"/>
+    <xacro:simple_link link_name="link0a" stl_name="rigid_link"/>
+	<xacro:simple_link link_name="link0b" stl_name="segment_base"/>
     <xacro:simple_link link_name="link1" stl_name="segment_link1"/>
     <xacro:simple_link link_name="link2" stl_name="segment_link2"/>
 	<joint name="segment_base" type="fixed">
-	<origin rpy="0 0 1.348574" xyz="-0.072698 -0.0085 -0.10417"/>
+	<origin rpy="0 0 1.348574" xyz="-0.1218 0.03 -0.11"/>
 		<parent link="chair_link2"/>
-		<child link="link0"/>
-	</joint>
-    <xacro:segment_joints joint_num="0" parent_link="link0" child_link="link1">
+		<child link="link0a"/>
+	</joint>
+    <xacro:segment_joints joint_num="b" parent_link="link0a" child_link="link0b">
+        <origin rpy="0.0 0.0 0.0" xyz="${joint_0_x} ${joint_0_y} ${joint_0_z}"/>
+        <axis xyz="-1.0 0.0 0.0"/>
+    </xacro:segment_joints>
+    <xacro:segment_joints joint_num="0" parent_link="link0b" child_link="link1">
         <origin rpy="0.0 0.0 0.0" xyz="${joint_0_x} ${joint_0_y} ${joint_0_z}"/>
         <axis xyz="-1.0 0.0 0.0"/>
@@ -171,5 +176,5 @@
     </xacro:segment_joints>
 <!-- Second segment (test) -->
-    <xacro:simple_link link_name="link3" stl_name="segment_base"/>
+    <!-- <xacro:simple_link link_name="link3" stl_name="segment_base"/>
     <xacro:simple_link link_name="link4" stl_name="segment_link1"/>
     <xacro:simple_link link_name="link5" stl_name="segment_link2"/>
@@ -186,7 +191,7 @@
         <origin rpy="0.0 0.0 0.0" xyz="${joint_1_x} ${joint_1_y} ${joint_1_z}"/>
         <axis xyz="0.0 0.0 1.0"/>
-    </xacro:segment_joints>
+    </xacro:segment_joints> -->
 <!-- Third segment (test) -->
-    <xacro:simple_link link_name="link6" stl_name="segment_base"/>
+    <!-- <xacro:simple_link link_name="link6" stl_name="segment_base"/>
     <xacro:simple_link link_name="link7" stl_name="segment_link1"/>
     <xacro:simple_link link_name="link8" stl_name="segment_link2"/>
@@ -203,7 +208,7 @@
         <origin rpy="0.0 0.0 0.0" xyz="${joint_1_x} ${joint_1_y} ${joint_1_z}"/>
         <axis xyz="0.0 0.0 1.0"/>
-    </xacro:segment_joints>
+    </xacro:segment_joints> -->
 <!-- Fourth segment (test) -->
-    <xacro:simple_link link_name="link9" stl_name="segment_base"/>
+    <!-- <xacro:simple_link link_name="link9" stl_name="segment_base"/>
     <xacro:simple_link link_name="link10" stl_name="segment_link1"/>
     <xacro:simple_link link_name="link11" stl_name="segment_link2"/>
@@ -220,7 +225,7 @@
         <origin rpy="0.0 0.0 0.0" xyz="${joint_1_x} ${joint_1_y} ${joint_1_z}"/>
         <axis xyz="0.0 0.0 1.0"/>
-    </xacro:segment_joints>
+    </xacro:segment_joints> -->
 <!-- Fifth segment (test) -->
-    <xacro:simple_link link_name="link12" stl_name="segment_base"/>
+    <!-- <xacro:simple_link link_name="link12" stl_name="segment_base"/>
     <xacro:simple_link link_name="link13" stl_name="segment_link1"/>
     <xacro:simple_link link_name="link14" stl_name="segment_link2"/>
@@ -237,5 +242,5 @@
         <origin rpy="0.0 0.0 0.0" xyz="${joint_1_x} ${joint_1_y} ${joint_1_z}"/>
         <axis xyz="0.0 0.0 1.0"/>
-    </xacro:segment_joints>
+    </xacro:segment_joints> -->
 	<!--
 		 Gazebo plugins:

Commit message: lined-up rigid link with segment base

File: urdf_stuff/src/wheelchair/robot.urdf.xacro (robot description, xacro)
@@ -164,5 +164,5 @@
 	</joint>
     <xacro:segment_joints joint_num="b" parent_link="link0a" child_link="link0b">
-        <origin rpy="0.0 0.0 0.0" xyz="${joint_0_x} ${joint_0_y} ${joint_0_z}"/>
+        <origin rpy="0.0 0.0 0.0" xyz="${joint_0_x-0.07} ${joint_0_y+0.013} ${joint_0_z-0.023}"/>
         <axis xyz="-1.0 0.0 0.0"/>
     </xacro:segment_joints>

Commit message: xacro for rigid link connection to segment base

File: urdf_stuff/src/wheelchair/robot.urdf.xacro (robot description, xacro)
@@ -147,4 +147,19 @@
     <!--*********************************************************************************-->
 </xacro:macro>
+<xacro:macro name="rigid_link" params="joint1 joint2 link1 link2 link3">
+<!--*********************************************************************************-->
+	<!-- Rigid link block -->
+	<joint name="${joint1}" type="fixed">
+	<origin rpy="0 0 0" xyz="0.0 0.0768 -0.02"/>
+		<parent link="${link1}"/>
+		<child link="${link2}"/>
+	</joint>
+	<joint name="${joint2}" type="fixed">
+	<origin rpy="0 0 0" xyz="${joint_0_x-0.07} ${joint_0_y+0.013} ${joint_0_z-0.023}"/>
+		<parent link="${link2}"/>
+		<child link="${link3}"/>
+	</joint>
+	<!--*********************************************************************************-->
+</xacro:macro>
 <xacro:property name="joint_0_x" value="0.04316036512320408" />
 <xacro:property name="joint_0_y" value="0.04848245206563817" />
@@ -158,4 +173,5 @@
     <xacro:simple_link link_name="link1" stl_name="segment_link1"/>
     <xacro:simple_link link_name="link2" stl_name="segment_link2"/>
+	<!-- First rigid link joints -->
 	<joint name="segment_base" type="fixed">
 	<origin rpy="0 0 1.348574" xyz="-0.1218 0.03 -0.11"/>
@@ -163,8 +179,10 @@
 		<child link="link0a"/>
 	</joint>
-    <xacro:segment_joints joint_num="b" parent_link="link0a" child_link="link0b">
-        <origin rpy="0.0 0.0 0.0" xyz="${joint_0_x-0.07} ${joint_0_y+0.013} ${joint_0_z-0.023}"/>
-        <axis xyz="-1.0 0.0 0.0"/>
-    </xacro:segment_joints>
+	<joint name="jointb" type="fixed">
+	<origin rpy="0 0 0" xyz="${joint_0_x-0.07} ${joint_0_y+0.013} ${joint_0_z-0.023}"/>
+		<parent link="link0a"/>
+		<child link="link0b"/>
+	</joint>
+	<!-- segment joints -->
     <xacro:segment_joints joint_num="0" parent_link="link0b" child_link="link1">
         <origin rpy="0.0 0.0 0.0" xyz="${joint_0_x} ${joint_0_y} ${joint_0_z}"/>
@@ -176,5 +194,5 @@
     </xacro:segment_joints>
 <!-- Second segment (test) -->
-    <!-- <xacro:simple_link link_name="link3" stl_name="segment_base"/>
+    <xacro:simple_link link_name="link3" stl_name="segment_base"/>
     <xacro:simple_link link_name="link4" stl_name="segment_link1"/>
     <xacro:simple_link link_name="link5" stl_name="segment_link2"/>
@@ -191,15 +209,15 @@
         <origin rpy="0.0 0.0 0.0" xyz="${joint_1_x} ${joint_1_y} ${joint_1_z}"/>
         <axis xyz="0.0 0.0 1.0"/>
-    </xacro:segment_joints> -->
+    </xacro:segment_joints>
 <!-- Third segment (test) -->
-    <!-- <xacro:simple_link link_name="link6" stl_name="segment_base"/>
+	<!-- Segment #2 rigid link joints -->
+    <xacro:simple_link link_name="link6a" stl_name="rigid_link"/>
+	<xacro:simple_link link_name="link6b" stl_name="segment_base"/>
     <xacro:simple_link link_name="link7" stl_name="segment_link1"/>
     <xacro:simple_link link_name="link8" stl_name="segment_link2"/>
-	<joint name="third_segment_base" type="fixed">
-	    <origin rpy="0 0 0" xyz="-0.02661 ${joint_1_y-0.0145-0.005} -0.0153545"/>
-		<parent link="link5"/>
-		<child link="link6"/>
-	</joint>
-    <xacro:segment_joints joint_num="4" parent_link="link6" child_link="link7">
+	<!-- Segment #2 rigid link joints -->
+	<xacro:rigid_link joint1="jointc" joint2="jointd" link1="link5" link2="link6a" link3="link6b"/>
+	<!-- Segmen #2 joints -->
+    <xacro:segment_joints joint_num="4" parent_link="link6b" child_link="link7">
         <origin rpy="0.0 0.0 0.0" xyz="${joint_0_x} ${joint_0_y} ${joint_0_z}"/>
         <axis xyz="-1.0 0.0 0.0"/>
@@ -208,5 +226,5 @@
         <origin rpy="0.0 0.0 0.0" xyz="${joint_1_x} ${joint_1_y} ${joint_1_z}"/>
         <axis xyz="0.0 0.0 1.0"/>
-    </xacro:segment_joints> -->
+    </xacro:segment_joints>
 <!-- Fourth segment (test) -->
     <!-- <xacro:simple_link link_name="link9" stl_name="segment_base"/>

Commit message: setting up xacro for simplifying rigid-link + segment URDF

File: urdf_stuff/src/wheelchair/robot.urdf.xacro (robot description, xacro)
@@ -211,12 +211,12 @@
     </xacro:segment_joints>
 <!-- Third segment (test) -->
-	<!-- Segment #2 rigid link joints -->
+	<!-- Segment #3 rigid link joints -->
     <xacro:simple_link link_name="link6a" stl_name="rigid_link"/>
 	<xacro:simple_link link_name="link6b" stl_name="segment_base"/>
     <xacro:simple_link link_name="link7" stl_name="segment_link1"/>
     <xacro:simple_link link_name="link8" stl_name="segment_link2"/>
-	<!-- Segment #2 rigid link joints -->
+	<!-- Segment #3 rigid link joints -->
 	<xacro:rigid_link joint1="jointc" joint2="jointd" link1="link5" link2="link6a" link3="link6b"/>
-	<!-- Segmen #2 joints -->
+	<!-- Segmen #3 joints -->
     <xacro:segment_joints joint_num="4" parent_link="link6b" child_link="link7">
         <origin rpy="0.0 0.0 0.0" xyz="${joint_0_x} ${joint_0_y} ${joint_0_z}"/>
@@ -228,8 +228,8 @@
     </xacro:segment_joints>
 <!-- Fourth segment (test) -->
-    <!-- <xacro:simple_link link_name="link9" stl_name="segment_base"/>
+	<xacro:simple_link link_name="link9" stl_name="segment_base"/>
     <xacro:simple_link link_name="link10" stl_name="segment_link1"/>
     <xacro:simple_link link_name="link11" stl_name="segment_link2"/>
-	<joint name="fourth_segment_base" type="fixed">
+	<joint name="third_segment_base" type="fixed">
 	    <origin rpy="0 0 0" xyz="-0.02661 ${joint_1_y-0.0145-0.005} -0.0153545"/>
 		<parent link="link8"/>
@@ -243,7 +243,7 @@
         <origin rpy="0.0 0.0 0.0" xyz="${joint_1_x} ${joint_1_y} ${joint_1_z}"/>
         <axis xyz="0.0 0.0 1.0"/>
-    </xacro:segment_joints> -->
+    </xacro:segment_joints>
 <!-- Fifth segment (test) -->
-    <!-- <xacro:simple_link link_name="link12" stl_name="segment_base"/>
+    <xacro:simple_link link_name="link12" stl_name="segment_base"/>
     <xacro:simple_link link_name="link13" stl_name="segment_link1"/>
     <xacro:simple_link link_name="link14" stl_name="segment_link2"/>
@@ -260,5 +260,5 @@
         <origin rpy="0.0 0.0 0.0" xyz="${joint_1_x} ${joint_1_y} ${joint_1_z}"/>
         <axis xyz="0.0 0.0 1.0"/>
-    </xacro:segment_joints> -->
+    </xacro:segment_joints>
 	<!--
 		 Gazebo plugins:
