Commit message: Automated appending to manipulator chain using xacro

File: urdf_stuff/src/wheelchair/robot.urdf.xacro (robot description, xacro)
@@ -93,7 +93,6 @@
 <!-- ***************** -->
 <!-- "xacro inorder SARA.xacro > SARA.urdf" -->
+<!--********************************************************************************************************-->
 <xacro:macro name="simple_link" params="link_name stl_name">
-    <!-- ${link_name} -->
-    <!--*********************************************************************************-->
     <link name="${link_name}">
         <inertial>
@@ -122,9 +121,9 @@
         <dampingFactor>0.005</dampingFactor>
     </gazebo>
-    <!--*********************************************************************************-->
-</xacro:macro>
+</xacro:macro>
+<!--********************************************************************************************************-->
+<!--********************************************************************************************************-->
 <xacro:macro name="segment_joints" params="joint_num parent_link child_link *origin *axis">
     <!-- joint${joint_num#} -->
-    <!--*********************************************************************************-->
 	<joint name="joint${joint_num#}" type="revolute">
 		<parent link="${parent_link}"/>
@@ -145,9 +144,10 @@
 		</actuator>
 	</transmission>
-    <!--*********************************************************************************-->
-</xacro:macro>
+</xacro:macro>
+<!--********************************************************************************************************-->
+<!-- *********************************************** -->
+<!-- Defines joints and link of a single rigid joint -->
+<!--********************************************************************************************************-->
 <xacro:macro name="rigid_link" params="joint1 joint2 link1 link2 link3">
-<!--*********************************************************************************-->
-	<!-- Rigid link block -->
 	<joint name="${joint1}" type="fixed">
 	<origin rpy="0 0 0" xyz="0.0 0.0768 -0.02"/>
@@ -160,6 +160,7 @@
 		<child link="${link3}"/>
 	</joint>
-	<!--*********************************************************************************-->
-</xacro:macro>
+</xacro:macro>
+<!--********************************************************************************************************-->
+<!-- Joint frame pose parameters -->
 <xacro:property name="joint_0_x" value="0.04316036512320408" />
 <xacro:property name="joint_0_y" value="0.04848245206563817" />
@@ -168,115 +169,98 @@
 <xacro:property name="joint_1_y" value="0.040054000000004225" />
 <xacro:property name="joint_1_z" value="-0.01210000000000057" />
-<!-- First segment -->
-    <xacro:simple_link link_name="link0a" stl_name="rigid_link"/>
-	<xacro:simple_link link_name="link0b" stl_name="segment_base"/>
-    <xacro:simple_link link_name="link1" stl_name="segment_link1"/>
-    <xacro:simple_link link_name="link2" stl_name="segment_link2"/>
-	<!-- First rigid link joints -->
-	<joint name="segment_base" type="fixed">
-	<origin rpy="0 0 1.348574" xyz="-0.1218 0.03 -0.11"/>
-		<parent link="chair_link2"/>
-		<child link="link0a"/>
-	</joint>
-	<joint name="jointb" type="fixed">
-	<origin rpy="0 0 0" xyz="${joint_0_x-0.07} ${joint_0_y+0.013} ${joint_0_z-0.023}"/>
-		<parent link="link0a"/>
-		<child link="link0b"/>
-	</joint>
-	<!-- segment joints -->
-    <xacro:segment_joints joint_num="0" parent_link="link0b" child_link="link1">
+<!-- Manipulator joint and link element coutners -->
+<xacro:property name="arm_joint_count" value="0"/>
+<xacro:property name="arm_link_count" value="0"/>
+<!-- ************************* -->
+<!-- 1 Rigid link + 2 Segments -->
+<!--********************************************************************************************************-->
+<xacro:macro name="L1S2" params="LinkID JointID parent is_manipulator_base">
+	<!-- Defining links -->
+    <xacro:simple_link link_name="link${LinkID}a" stl_name="rigid_link"/>
+	<xacro:simple_link link_name="link${LinkID}b" stl_name="segment_base"/>
+    <xacro:simple_link link_name="link${LinkID+1}" stl_name="segment_link1"/>
+    <xacro:simple_link link_name="link${LinkID+2}" stl_name="segment_link2"/>
+	<xacro:simple_link link_name="link${LinkID+3}" stl_name="segment_base"/>
+    <xacro:simple_link link_name="link${LinkID+4}" stl_name="segment_link1"/>
+    <xacro:simple_link link_name="link${LinkID+5}" stl_name="segment_link2"/>
+	<!-- Rigid link joints -->
+		<!-- Handles case where manipulator connects directly to the shoulder -->
+		<xacro:if value="${is_manipulator_base}">
+			<joint name="fixed_proximal${JointID}" type="fixed">
+			<origin rpy="0 0 1.348574" xyz="-0.1218 0.03 -0.11"/>
+				<parent link="${parent}"/>
+				<child link="link${LinkID}a"/>
+			</joint>
+			<joint name="fixed_distal${JointID}" type="fixed">
+			<origin rpy="0 0 0" xyz="${joint_0_x-0.07} ${joint_0_y+0.013} ${joint_0_z-0.023}"/>
+				<parent link="link${LinkID}a"/>
+				<child link="link${LinkID}b"/>
+			</joint>
+		</xacro:if>
+		<!-- Handles case where rigid link does not connect directly to the shoulder -->
+		<xacro:unless value="${is_manipulator_base}">
+			<joint name="fixed_proximal${JointID}" type="fixed">
+			<origin rpy="0 0 0" xyz="0.0 0.0768 -0.02"/>
+				<parent link="${parent}"/>
+				<child link="link${LinkID}a"/>
+			</joint>
+			<joint name="fixed_distal${JointID}" type="fixed">
+			<origin rpy="0 0 0" xyz="${joint_0_x-0.07} ${joint_0_y+0.013} ${joint_0_z-0.023}"/>
+				<parent link="link${LinkID}a"/>
+				<child link="link${LinkID}b"/>
+			</joint>
+		</xacro:unless>
+	<!-- First Segment joints -->
+    <xacro:segment_joints joint_num="${JointID}" parent_link="link${LinkID}b" child_link="link${LinkID+1}">
         <origin rpy="0.0 0.0 0.0" xyz="${joint_0_x} ${joint_0_y} ${joint_0_z}"/>
         <axis xyz="-1.0 0.0 0.0"/>
     </xacro:segment_joints>
-    <xacro:segment_joints joint_num="1" parent_link="link1" child_link="link2">
+    <xacro:segment_joints joint_num="${JointID+1}" parent_link="link${LinkID+1}" child_link="link${LinkID+2}">
         <origin rpy="0.0 0.0 0.0" xyz="${joint_1_x} ${joint_1_y} ${joint_1_z}"/>
         <axis xyz="0.0 0.0 1.0"/>
     </xacro:segment_joints>
-<!-- Second segment (test) -->
-    <xacro:simple_link link_name="link3" stl_name="segment_base"/>
-    <xacro:simple_link link_name="link4" stl_name="segment_link1"/>
-    <xacro:simple_link link_name="link5" stl_name="segment_link2"/>
-	<joint name="second_segment_base" type="fixed">
+	<!-- Fixed joint between two segments -->
+	<joint name="segment_base${JointID}" type="fixed">
 	    <origin rpy="0 0 0" xyz="-0.02661 ${joint_1_y-0.0145-0.005} -0.0153545"/>
-		<parent link="link2"/>
-		<child link="link3"/>
-	</joint>
-    <xacro:segment_joints joint_num="2" parent_link="link3" child_link="link4">
+		<parent link="link${LinkID+2}"/>
+		<child link="link${LinkID+3}"/>
+	</joint>
+	<!-- Second segment joints -->
+    <xacro:segment_joints joint_num="${JointID+2}" parent_link="link${LinkID+3}" child_link="link${LinkID+4}">
         <origin rpy="0.0 0.0 0.0" xyz="${joint_0_x} ${joint_0_y} ${joint_0_z}"/>
         <axis xyz="-1.0 0.0 0.0"/>
     </xacro:segment_joints>
-    <xacro:segment_joints joint_num="3" parent_link="link4" child_link="link5">
+    <xacro:segment_joints joint_num="${JointID+3}" parent_link="link${LinkID+4}" child_link="link${LinkID+5}">
         <origin rpy="0.0 0.0 0.0" xyz="${joint_1_x} ${joint_1_y} ${joint_1_z}"/>
         <axis xyz="0.0 0.0 1.0"/>
     </xacro:segment_joints>
-<!-- Third segment (test) -->
-	<!-- Segment #3 rigid link joints -->
-    <xacro:simple_link link_name="link6a" stl_name="rigid_link"/>
-	<xacro:simple_link link_name="link6b" stl_name="segment_base"/>
-    <xacro:simple_link link_name="link7" stl_name="segment_link1"/>
-    <xacro:simple_link link_name="link8" stl_name="segment_link2"/>
-	<!-- Segment #3 rigid link joints -->
-	<xacro:rigid_link joint1="jointc" joint2="jointd" link1="link5" link2="link6a" link3="link6b"/>
-	<!-- Segmen #3 joints -->
-    <xacro:segment_joints joint_num="4" parent_link="link6b" child_link="link7">
-        <origin rpy="0.0 0.0 0.0" xyz="${joint_0_x} ${joint_0_y} ${joint_0_z}"/>
-        <axis xyz="-1.0 0.0 0.0"/>
-    </xacro:segment_joints>
-    <xacro:segment_joints joint_num="5" parent_link="link7" child_link="link8">
-        <origin rpy="0.0 0.0 0.0" xyz="${joint_1_x} ${joint_1_y} ${joint_1_z}"/>
-        <axis xyz="0.0 0.0 1.0"/>
-    </xacro:segment_joints>
-<!-- Fourth segment (test) -->
-	<xacro:simple_link link_name="link9" stl_name="segment_base"/>
-    <xacro:simple_link link_name="link10" stl_name="segment_link1"/>
-    <xacro:simple_link link_name="link11" stl_name="segment_link2"/>
-	<joint name="third_segment_base" type="fixed">
-	    <origin rpy="0 0 0" xyz="-0.02661 ${joint_1_y-0.0145-0.005} -0.0153545"/>
-		<parent link="link8"/>
-		<child link="link9"/>
-	</joint>
-    <xacro:segment_joints joint_num="6" parent_link="link9" child_link="link10">
-        <origin rpy="0.0 0.0 0.0" xyz="${joint_0_x} ${joint_0_y} ${joint_0_z}"/>
-        <axis xyz="-1.0 0.0 0.0"/>
-    </xacro:segment_joints>
-    <xacro:segment_joints joint_num="7" parent_link="link10" child_link="link11">
-        <origin rpy="0.0 0.0 0.0" xyz="${joint_1_x} ${joint_1_y} ${joint_1_z}"/>
-        <axis xyz="0.0 0.0 1.0"/>
-    </xacro:segment_joints>
-<!-- Fifth segment (test) -->
-    <xacro:simple_link link_name="link12" stl_name="segment_base"/>
-    <xacro:simple_link link_name="link13" stl_name="segment_link1"/>
-    <xacro:simple_link link_name="link14" stl_name="segment_link2"/>
-	<joint name="fifth_segment_base" type="fixed">
-	    <origin rpy="0 0 0" xyz="-0.02661 ${joint_1_y-0.0145-0.005} -0.0153545"/>
-		<parent link="link11"/>
-		<child link="link12"/>
-	</joint>
-    <xacro:segment_joints joint_num="8" parent_link="link12" child_link="link13">
-        <origin rpy="0.0 0.0 0.0" xyz="${joint_0_x} ${joint_0_y} ${joint_0_z}"/>
-        <axis xyz="-1.0 0.0 0.0"/>
-    </xacro:segment_joints>
-    <xacro:segment_joints joint_num="9" parent_link="link13" child_link="link14">
-        <origin rpy="0.0 0.0 0.0" xyz="${joint_1_x} ${joint_1_y} ${joint_1_z}"/>
-        <axis xyz="0.0 0.0 1.0"/>
-    </xacro:segment_joints>
-	<!--
-		 Gazebo plugins:
-			ros_control
-			* Accepts new desired trajectories via follow_joint_trajectory, while joint_state_publisher publishes joint_states.
-			* Makes joints move.
-			joint_state_publisher
-			* Publish current state of each joint to a topic
-	-->
-	<gazebo>
-		<plugin name="control" filename="libgazebo_ros_control.so" >
-			<robotNamespace>/SARA</robotNamespace>
-		</plugin>
-		<plugin name="joint_state_publisher" filename="libgazebo_ros_joint_state_publisher.so" >
-			<jointName>joint0, joint1, joint2, joint3, joint4, joint5, joint6, joint7</jointName>
-			<updateRate>100.0</updateRate>
-			<alwaysOn>true</alwaysOn>
-			<!-- <robotNamespace>/SARA</robotNamespace> -->
-		</plugin>
-	</gazebo>
+</xacro:macro>
+<!--********************************************************************************************************-->
+<!-- L1S2 [1]-->
+<xacro:L1S2 LinkID="0" JointID="0" parent="chair_link2" is_manipulator_base="true"/>
+<!-- L1S2 [2]-->
+<xacro:L1S2 LinkID="6" JointID="4" parent="link5" is_manipulator_base="false"/>
+<!-- L1S2 [3]-->
+<xacro:L1S2 LinkID="13" JointID="9" parent="link11" is_manipulator_base="false"/>
+<!-- L1S2 [4]-->
+<xacro:L1S2 LinkID="20" JointID="14" parent="link17" is_manipulator_base="false"/>
+<!--
+		Gazebo plugins:
+		ros_control
+		* Accepts new desired trajectories via follow_joint_trajectory, while joint_state_publisher publishes joint_states.
+		* Makes joints move.
+		joint_state_publisher
+		* Publish current state of each joint to a topic
+-->
+<gazebo>
+	<plugin name="control" filename="libgazebo_ros_control.so" >
+		<robotNamespace>/SARA</robotNamespace>
+	</plugin>
+	<plugin name="joint_state_publisher" filename="libgazebo_ros_joint_state_publisher.so" >
+		<jointName>joint0, joint1, joint2, joint3, joint4, joint5, joint6, joint7</jointName>
+		<updateRate>100.0</updateRate>
+		<alwaysOn>true</alwaysOn>
+		<!-- <robotNamespace>/SARA</robotNamespace> -->
+	</plugin>
+</gazebo>
 </robot>
