Commit message: gazebo sim appears to be working

File: urdf_stuff/src/wheelchair/REACH.urdf.xacro (robot description, xacro)
@@ -1,18 +1,17 @@
 <?xml version="1.0" ?>
-<robot name="SARA" xmlns:xacro="http://www.ros.org/wiki/xacro">
-	<link name="base_link"/>
-	<joint name="set_worldaxis" type="fixed">
-		<origin rpy="1.570796326795 0 0" xyz="0.0 0.0 0.0"/>
-		<parent link="base_link"/>
+<robot name="REACH" xmlns:xacro="http://www.ros.org/wiki/xacro">
+	<link name="world"/>
+	<joint name="world_frame" type="fixed">
+		<origin rpy="1.570796326795 0 0" xyz="0.0 0.0 0.1"/>
+		<parent link="world"/>
 		<child link="chair_base"/>
 		<axis xyz="0 0 0"/>
-		<limit effort="0" lower="-1" upper="1" velocity="0"/>
 	</joint>
 	<link name="chair_base">
-		<inertial>
-			<origin rpy="0.0 0.0 0.0" xyz="0.0 0.0 0.0"/>
-			<mass value="0"/>
-			<inertia ixx="0" ixy="0" ixz="0" iyy="0" iyz="0" izz="0"/>
-		</inertial>
+        <inertial>
+            <origin rpy="0.0 0.0 0.0" xyz="0.0 0.0 0.0"/>
+            <mass value="0.2"/>
+            <inertia ixx="0.01" ixy="0.01" ixz="0.01" iyy="0.01" iyz="0.01" izz="0.1"/>
+        </inertial>
 		<visual>
 			<origin rpy="0.0 0.0 0.0" xyz="0.0 0.0 0.0"/>
@@ -32,9 +31,9 @@
 	</link>
 	<link name="chair_link1">
-		<inertial>
-			<origin rpy="0.0 0.0 0.0" xyz="0.0 0.0 0.0"/>
-			<mass value="0"/>
-			<inertia ixx="0" ixy="0" ixz="0" iyy="0" iyz="0" izz="0"/>
-		</inertial>
+        <inertial>
+            <origin rpy="0.0 0.0 0.0" xyz="0.0 0.0 0.0"/>
+            <mass value="0.2"/>
+            <inertia ixx="0.01" ixy="0.01" ixz="0.01" iyy="0.01" iyz="0.01" izz="0.01"/>
+        </inertial>
 		<visual>
 			<origin rpy="0.0 0.0 0.0" xyz="0.0 0.0 0.0"/>
@@ -54,9 +53,9 @@
 	</link>
 	<link name="chair_link2">
-		<inertial>
-			<origin rpy="0.0 0.0 0.0" xyz="0.0 0.0 0.0"/>
-			<mass value="0"/>
-			<inertia ixx="0" ixy="0" ixz="0" iyy="0" iyz="0" izz="0"/>
-		</inertial>
+        <inertial>
+            <origin rpy="0.0 0.0 0.0" xyz="0.0 0.0 0.0"/>
+            <mass value="0.2"/>
+            <inertia ixx="0.01" ixy="0.01" ixz="0.01" iyy="0.01" iyz="0.01" izz="0.01"/>
+        </inertial>
 		<visual>
 			<origin rpy="0.0 0.0 0.0" xyz="0.0 0.0 0.0"/>
@@ -75,22 +74,51 @@
 		</collision>
 	</link>
-	<joint name="chair_joint1" type="continuous">
+	<gazebo reference="chair_base">
+        <dampingFactor>0.005</dampingFactor>
+    </gazebo>
+	<gazebo reference="chair_link1">
+        <dampingFactor>0.005</dampingFactor>
+    </gazebo>
+	<gazebo reference="chair_link2">
+        <dampingFactor>0.005</dampingFactor>
+    </gazebo>
+	<joint name="chair_joint1" type="revolute">
 		<origin rpy="0.0 0.0 0.0" xyz="0.6162001603339797 0.9987983990460869 -0.10515639316991093"/>
 		<parent link="chair_base"/>
 		<child link="chair_link1"/>
 		<axis xyz="-0.9698848187392894 0.24356401227352137 0.00010151002393613432"/>
-		<limit effort="0" lower="-1" upper="1" velocity="0"/>
-	</joint>
-	<joint name="chair_joint2" type="continuous">
+		<limit effort="30" lower="-3.14159" upper="3.14159" velocity="1.0"/>
+	</joint>
+	<joint name="chair_joint2" type="revolute">
 		<origin rpy="0.0 0.0 0.0" xyz="-0.05333534440670149 0.013396020675043162 0.07950558261589771"/>
 		<parent link="chair_link1"/>
 		<child link="chair_link2"/>
 		<axis xyz="-0.00010466193655742605 -1.1955594058051162e-14 -0.99999999452302"/>
-		<limit effort="0" lower="-1" upper="1" velocity="0"/>
-	</joint>
+		<limit effort="30" lower="-3.14159" upper="3.14159" velocity="1.0"/>
+	</joint>
+    <transmission name="tran_chair_joint1">
+		<type>transmission_interface/SimpleTransmission</type>
+		<joint name="chair_joint1">
+			<hardwareInterface>hardware_interface/EffortJointInterface</hardwareInterface>
+		</joint>
+		<actuator name="tmotor_chair_joint1">
+			<hardwareInterface>hardware_interface/EffortJointInterface</hardwareInterface>
+            <mechanicalReduction>1</mechanicalReduction>
+		</actuator>
+	</transmission>
+    <transmission name="tran_chair_joint2">
+		<type>transmission_interface/SimpleTransmission</type>
+		<joint name="chair_joint2">
+			<hardwareInterface>hardware_interface/EffortJointInterface</hardwareInterface>
+		</joint>
+		<actuator name="tmotor_chair_joint2">
+			<hardwareInterface>hardware_interface/EffortJointInterface</hardwareInterface>
+            <mechanicalReduction>1</mechanicalReduction>
+		</actuator>
+	</transmission>
 <!-- ***************** -->
 <!-- Manipulator stuff -->
 <!-- ***************** -->
-<!-- "xacro inorder SARA.xacro > SARA.urdf" -->
+<!-- "xacro inorder REACH.xacro > REACH.urdf" -->
 <!--********************************************************************************************************-->
 <xacro:macro name="simple_link" params="link_name stl_name">
@@ -144,20 +172,4 @@
 		</actuator>
 	</transmission>
-</xacro:macro>
-<!--********************************************************************************************************-->
-<!-- *********************************************** -->
-<!-- Defines joints and link of a single rigid joint -->
-<!--********************************************************************************************************-->
-<xacro:macro name="rigid_link" params="joint1 joint2 link1 link2 link3">
-	<joint name="${joint1}" type="fixed">
-	<origin rpy="0 0 0" xyz="0.0 0.0768 -0.02"/>
-		<parent link="${link1}"/>
-		<child link="${link2}"/>
-	</joint>
-	<joint name="${joint2}" type="fixed">
-	<origin rpy="0 0 0" xyz="${joint_0_x-0.07} ${joint_0_y+0.013} ${joint_0_z-0.023}"/>
-		<parent link="${link2}"/>
-		<child link="${link3}"/>
-	</joint>
 </xacro:macro>
 <!--********************************************************************************************************-->
@@ -242,7 +254,7 @@
 <xacro:L1S2 LinkID="6" JointID="4" parent="link5" is_manipulator_base="false"/>
 <!-- L1S2 [3]-->
-<xacro:L1S2 LinkID="13" JointID="9" parent="link11" is_manipulator_base="false"/>
+<xacro:L1S2 LinkID="12" JointID="8" parent="link11" is_manipulator_base="false"/>
 <!-- L1S2 [4]-->
-<xacro:L1S2 LinkID="20" JointID="14" parent="link18" is_manipulator_base="false"/>
+<xacro:L1S2 LinkID="18" JointID="12" parent="link17" is_manipulator_base="false"/>
 <!--
 		Gazebo plugins:
@@ -255,5 +267,5 @@
 <gazebo>
 	<plugin name="control" filename="libgazebo_ros_control.so" >
-		<robotNamespace>/SARA</robotNamespace>
+		<robotNamespace>/REACH</robotNamespace>
 	</plugin>
 	<plugin name="joint_state_publisher" filename="libgazebo_ros_joint_state_publisher.so" >
@@ -261,5 +273,5 @@
 		<updateRate>100.0</updateRate>
 		<alwaysOn>true</alwaysOn>
-		<!-- <robotNamespace>/SARA</robotNamespace> -->
+		<!-- <robotNamespace>/REACH</robotNamespace> -->
 	</plugin>
 </gazebo>
